File: ESP32-Sentinel-Kinetic-Wireless-Dongle.kicad_sch (KiCad schematic)
At the start: 81 parts, among them J1 RJ9, J2 RJ9, J3 Conn_01x06_Pin, J4 Conn_01x01_Pin, J5 Conn_01x04_Pin, J6 Conn_01x06_Pin, J7 Conn_02x06_Odd_Even, J8 Conn_01x07_Socket, Q1 SS8050, SW1 SW_Push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

Commit message: Updated LCSC numbers
Parts:
- Q1: LCSC (none) -> C431710
- U2: LCSC (none) -> C71035
- U4: now not fitted; now left out of the parts list
- U7: LCSC (none) -> C61063
